File: schematic/power.sch (KiCad schematic (older format))
At the start: 56 parts, among them J6 Conn_01x06, J7 Conn_01x03, U6 BD9E302EFJ, U7 BD9E302EFJ, U8 BD9E302EFJ

Commit message: Revert "Updated to kicad 5.0.0"
This reverts commit 6c14fa6c8e6361c9b9ee4065803a5a63755fc6a7.
Parts:
- C62, C63, C64, C65, C66, C67, C70, C71, C72, C73, C74, C75, C76, C77, C78, C79, C80, C81, C82, C83, C84, C85, C86, C87, C88, C89, C90, C91, C92: symbol Device:C -> C
- C68, C69: symbol Device:CP -> CP
- D1, D2, D3: symbol Device:D_Schottky -> D_Schottky
- F1, F2, F3: symbol Device:Fuse -> Fuse
- J6: symbol Connector_Generic:Conn_01x06 -> Conn_01x06
- J7: symbol Connector_Generic:Conn_01x03 -> Conn_01x03
- L17, L18: symbol Device:L_Core_Ferrite -> L_Core_Ferrite
- L19, L20, L21: symbol Device:L -> L
- R19, R20, R21, R22, R23, R24, R25, R26, R27: symbol Device:R -> R
- U6, U7, U8: symbol bd9e302efj:BD9E302EFJ -> BD9E302EFJ

Commit message: Updated to kicad 5.0.0
Parts:
- C62, C63, C64, C65, C66, C67, C70, C71, C72, C73, C74, C75, C76, C77, C78, C79, C80, C81, C82, C83, C84, C85, C86, C87, C88, C89, C90, C91, C92: symbol C -> Device:C
- C68, C69: symbol CP -> Device:CP
- D1, D2, D3: symbol D_Schottky -> Device:D_Schottky
- F1, F2, F3: symbol Fuse -> Device:Fuse
- J6: symbol Conn_01x06 -> Connector_Generic:Conn_01x06
- J7: symbol Conn_01x03 -> Connector_Generic:Conn_01x03
- L17, L18: symbol L_Core_Ferrite -> Device:L_Core_Ferrite
- L19, L20, L21: symbol L -> Device:L
- R19, R20, R21, R22, R23, R24, R25, R26, R27: symbol R -> Device:R
- U6, U7, U8: symbol BD9E302EFJ -> bd9e302efj:BD9E302EFJ
