File: schematic/power.sch (KiCad schematic (older format))
At the start: 56 parts, among them J6 Conn_01x06, J7 Conn_01x03, U6 BD9E302EFJ, U7 BD9E302EFJ, U8 BD9E302EFJ

Commit message: Removed some components
Parts:
- L19, L20, L21: footprint Inductors_SMD:L_Taiyo-Yuden_NR-60xx_HandSoldering -> Inductor_SMD:L_Taiyo-Yuden_NR-60xx

Commit message: Added logo's and stm32 capacitors
Parts:
- L19, L20, L21: footprint Inductor_SMD:L_Taiyo-Yuden_NR-60xx -> Inductors_SMD:L_Taiyo-Yuden_NR-60xx

Commit message: Updated to kicad v5
Parts:
- C62, C63, C64, C65, C66, C67, C70, C71, C72, C73, C74, C75, C76, C77, C78, C79, C80, C81, C82, C83, C84, C85, C86, C87, C88, C89, C90, C91, C92: symbol C -> schematic-rescue:C
- C68, C69: symbol CP -> schematic-rescue:CP
- D1, D2, D3: symbol D_Schottky -> schematic-rescue:D_Schottky
- F1, F2, F3: symbol Fuse -> schematic-rescue:Fuse
- J6: symbol Conn_01x06 -> schematic-rescue:Conn_01x06
- J7: symbol Conn_01x03 -> schematic-rescue:Conn_01x03
- L17, L18: symbol L_Core_Ferrite -> schematic-rescue:L_Core_Ferrite
- L19, L20, L21: symbol L -> schematic-rescue:L
- R19, R20, R21, R22, R23, R24, R25, R26, R27: symbol R -> schematic-rescue:R
- U6, U7, U8: symbol BD9E302EFJ -> bd9e302efj:BD9E302EFJ

Commit message: Moved to L6470 driver
Parts:
- C62, C63, C64, C65, C66, C67, C70, C71, C75, C76, C77, C78, C79, C80, C81, C82, C83, C84, C85, C86: footprint Capacitors_SMD:C_0603 -> Capacitor_SMD:C_0603_1608Metric; symbol schematic-rescue:C -> Device:C
- C68, C69: footprint Capacitors_SMD:CP_Elec_8x10 -> Capacitor_SMD:CP_Elec_8x10; symbol schematic-rescue:CP -> Device:CP
- C72, C73, C74, C87, C88, C89, C90, C91, C92: footprint Capacitors_SMD:C_1206 -> Capacitor_SMD:C_1206_3216Metric; symbol schematic-rescue:C -> Device:C
- D1, D2, D3: footprint Diodes_SMD:D_SMA -> Diode_SMD:D_SMA; symbol schematic-rescue:D_Schottky -> Device:D_Schottky
- F1, F2, F3: symbol schematic-rescue:Fuse -> Device:Fuse
- J6: symbol schematic-rescue:Conn_01x06 -> Connector_Generic:Conn_01x06
- J7: symbol schematic-rescue:Conn_01x03 -> Connector_Generic:Conn_01x03
- L17, L18: footprint Inductors_SMD:L_1806 -> Inductor_SMD:L_1806_4516Metric; symbol schematic-rescue:L_Core_Ferrite -> Device:L_Core_Ferrite
- L19, L20, L21: footprint Inductors_SMD:L_Taiyo-Yuden_NR-60xx -> Inductor_SMD:L_Taiyo-Yuden_NR-60xx; symbol schematic-rescue:L -> Device:L
- R19, R20, R21, R22, R23, R24, R25, R26, R27: footprint Resistors_SMD:R_0603 -> Resistor_SMD:R_0603_1608Metric; symbol schematic-rescue:R -> Device:R
