File: schematic/Mosfet.sch (KiCad schematic (older format))
At the start: 35 parts, among them J10 Conn_01x03, J8 Screw_Terminal_01x02, J9 Conn_01x03, Q1 PSMN1R7-30YL, Q2 PSMN1R7-30YL, Q3 NCV8402, Q4 NCV8402

Commit message: Updated to kicad 5.0.0
Parts:
- C93, C94: symbol C -> Device:C
- D10, D11: symbol D_Schottky_x2_Serial_AKC -> Device:D_Schottky_x2_Serial_AKC
- D4, D5: symbol D_Schottky -> Device:D_Schottky
- D6, D7, D8, D9: symbol LED -> Device:LED
- J10, J9: symbol Conn_01x03 -> Connector_Generic:Conn_01x03
- J8: symbol Screw_Terminal_01x02 -> Connector_Specialized:Screw_Terminal_01x02
- Q1, Q2: symbol PSMN1 -> psmn1:PSMN1
- Q3, Q4: symbol Q_NMOS_GDSD -> Device:Q_NMOS_GDSD
- R28, R29, R30, R31, R32, R33, R34, R35, R36, R37, R38, R39, R40, R41, R42, R43, R44, R45: symbol R -> Device:R

Commit message: Revert "Updated to kicad 5.0.0"
This reverts commit 6c14fa6c8e6361c9b9ee4065803a5a63755fc6a7.
Parts:
- C93, C94: symbol Device:C -> C
- D10, D11: symbol Device:D_Schottky_x2_Serial_AKC -> D_Schottky_x2_Serial_AKC
- D4, D5: symbol Device:D_Schottky -> D_Schottky
- D6, D7, D8, D9: symbol Device:LED -> LED
- J10, J9: symbol Connector_Generic:Conn_01x03 -> Conn_01x03
- J8: symbol Connector_Specialized:Screw_Terminal_01x02 -> Screw_Terminal_01x02
- Q1, Q2: symbol psmn1:PSMN1 -> PSMN1
- Q3, Q4: symbol Device:Q_NMOS_GDSD -> Q_NMOS_GDSD
- R28, R29, R30, R31, R32, R33, R34, R35, R36, R37, R38, R39, R40, R41, R42, R43, R44, R45: symbol Device:R -> R
