File: schematic/Mosfet.sch (KiCad schematic (older format))
At the start: 27 parts, among them J10 Conn_01x03, J8 Screw_Terminal_01x02, J9 Conn_01x03, Q1 PSMN1R7-30YL, Q2 PSMN1R7-30YL, Q3 NCV8402, Q4 NCV8402

Commit message: Moved to L6470 driver
Parts:
- D4, D5: footprint Diodes_SMD:D_SMA -> Diode_SMD:D_SMA; symbol schematic-rescue:D_Schottky -> Device:D_Schottky
- D6, D7, D8, D9: footprint LEDs:LED_0805 -> LED_SMD:LED_0805_2012Metric; symbol schematic-rescue:LED -> Device:LED
- J10, J9: symbol schematic-rescue:Conn_01x03 -> Connector_Generic:Conn_01x03
- Q3, Q4: footprint TO_SOT_Packages_SMD:SOT-223 -> Package_TO_SOT_SMD:SOT-223; symbol schematic-rescue:Q_NMOS_GDSD -> Device:Q_NMOS_GDSD
- R28, R29, R30, R31, R32, R33, R34, R35, R36, R37, R38, R39, R44, R45: footprint Resistors_SMD:R_0603 -> Resistor_SMD:R_0603_1608Metric; symbol schematic-rescue:R -> Device:R
