File: schematic/sensors.sch (KiCad schematic (older format))
At the start: 41 parts, among them J11 Conn_01x02, J12 Conn_01x02, J13 Conn_01x02, J14 Conn_01x02, J15 Conn_01x02, J16 Conn_01x02, J17 Conn_01x04, SW2 SW_DIP_x03

Commit message: Updated to kicad 5.0.0
Parts:
- C95, C96, C97, C98, C99: symbol C -> Device:C
- D12, D13, D14, D15: symbol D_Schottky_x2_Serial_AKC -> Device:D_Schottky_x2_Serial_AKC
- D16: symbol D_Zener -> Device:D_Zener
- D17, D18, D19: symbol D -> Device:D
- J11, J12, J13, J14, J15, J16: symbol Conn_01x02 -> Connector_Generic:Conn_01x02
- J17: symbol Conn_01x04 -> Connector_Generic:Conn_01x04
- R46, R47, R48, R49, R50, R51, R52, R53, R54, R55, R56, R57, R58, R59, R60, R61, R62, R63, R64, R65: symbol R -> Device:R
- SW2: symbol SW_DIP_x03 -> Switch:SW_DIP_x03

Commit message: Revert "Updated to kicad 5.0.0"
This reverts commit 6c14fa6c8e6361c9b9ee4065803a5a63755fc6a7.
Parts:
- C95, C96, C97, C98, C99: symbol Device:C -> C
- D12, D13, D14, D15: symbol Device:D_Schottky_x2_Serial_AKC -> D_Schottky_x2_Serial_AKC
- D16: symbol Device:D_Zener -> D_Zener
- D17, D18, D19: symbol Device:D -> D
- J11, J12, J13, J14, J15, J16: symbol Connector_Generic:Conn_01x02 -> Conn_01x02
- J17: symbol Connector_Generic:Conn_01x04 -> Conn_01x04
- R46, R47, R48, R49, R50, R51, R52, R53, R54, R55, R56, R57, R58, R59, R60, R61, R62, R63, R64, R65: symbol Device:R -> R
- SW2: symbol Switch:SW_DIP_x03 -> SW_DIP_x03
