File: schematic/sensors.sch (KiCad schematic (older format))
At the start: 41 parts, among them J11 Conn_01x02, J12 Conn_01x02, J13 Conn_01x02, J14 Conn_01x02, J15 Conn_01x02, J16 Conn_01x02, J17 Conn_01x04, SW2 SW_DIP_x03

Commit message: Updated to kicad v5
Parts:
- C95, C96, C97, C98, C99: symbol C -> schematic-rescue:C
- D12, D13, D14, D15: symbol D_Schottky_x2_Serial_AKC -> schematic-rescue:D_Schottky_x2_Serial_AKC
- D16: symbol D_Zener -> schematic-rescue:D_Zener
- D17, D18, D19: symbol D -> schematic-rescue:D
- J11, J12, J13, J14, J15, J16: symbol Conn_01x02 -> schematic-rescue:Conn_01x02
- J17: symbol Conn_01x04 -> schematic-rescue:Conn_01x04
- R46, R47, R48, R49, R50, R51, R52, R53, R54, R55, R56, R57, R58, R59, R60, R61, R62, R63, R64, R65: symbol R -> schematic-rescue:R
- SW2: symbol SW_DIP_x03 -> schematic-rescue:SW_DIP_x03

Commit message: Moved to L6470 driver
Parts:
- C95, C96, C97, C98, C99: footprint Capacitors_SMD:C_0603 -> Capacitor_SMD:C_0603_1608Metric; symbol schematic-rescue:C -> Device:C
- D12, D13, D14, D15: value BAT54SW -> BAV99,215; footprint TO_SOT_Packages_SMD:SOT-323_SC-70 -> Package_TO_SOT_SMD:SOT-323_SC-70; symbol schematic-rescue:D_Schottky_x2_Serial_AKC -> Device:D_Schottky_x2_Serial_AKC
- D16: footprint Diodes_SMD:D_SOD-123 -> Diode_SMD:D_SOD-123; symbol schematic-rescue:D_Zener -> Device:D_Zener
- D17, D18, D19: footprint Diodes_SMD:D_MiniMELF -> Diode_SMD:D_MiniMELF; symbol schematic-rescue:D -> Device:D
- J11, J12, J13, J14, J15, J16: footprint Socket_Strips:Socket_Strip_Straight_1x02_Pitch2.54mm -> Connector_PinHeader_2.54mm:PinHeader_1x02_P2.54mm_Vertical; symbol schematic-rescue:Conn_01x02 -> Connector_Generic:Conn_01x02
- J17: footprint Socket_Strips:Socket_Strip_Straight_1x04_Pitch2.54mm -> Connector_PinHeader_2.54mm:PinHeader_1x04_P2.54mm_Vertical; symbol schematic-rescue:Conn_01x04 -> Connector_Generic:Conn_01x04
- R46, R47, R48, R49, R50, R51, R52, R53, R54, R55, R56, R57, R58, R59, R60, R61, R62, R63, R64, R65: footprint Resistors_SMD:R_0603 -> Resistor_SMD:R_0603_1608Metric; symbol schematic-rescue:R -> Device:R
- SW2: symbol schematic-rescue:SW_DIP_x03 -> Switch:SW_DIP_x03
