File: schematic/aref.sch (KiCad schematic (older format))
At the start: 15 parts

Commit message: Updated to kicad 5.0.0
Parts:
- C100, C101, C102, C103, C104, C105: symbol C -> Device:C
- R66, R67, R68, R69, R70, R71, R72, R73, R74: symbol R -> Device:R
Changed lines of the file:
@@
-EESchema Schematic File Version 2
-LIBS:74xgxx
-LIBS:74xx
-LIBS:ac-dc
-LIBS:actel
-LIBS:adc-dac
-LIBS:allegro
-LIBS:Altera
-LIBS:analog_devices
-LIBS:analog_switches
-LIBS:atmel
-LIBS:audio
-LIBS:battery_management
-LIBS:bbd
-LIBS:bosch
-LIBS:brooktre
-LIBS:cmos4000
-LIBS:cmos_ieee
-LIBS:conn
-LIBS:contrib
-LIBS:cypress
-LIBS:dc-dc
-LIBS:device
-LIBS:digital-audio
-LIBS:diode
-LIBS:display
-LIBS:dsp
-LIBS:elec-unifil
-LIBS:ESD_Protection
-LIBS:ftdi
-LIBS:gennum
-LIBS:graphic_symbols
-LIBS:hc11
-LIBS:infineon
-LIBS:intel
-LIBS:interface
-LIBS:intersil
-LIBS:ir
-LIBS:Lattice
-LIBS:leds
-LIBS:LEM
-LIBS:linear
-LIBS:logic_programmable
-LIBS:maxim
-LIBS:mechanical
-LIBS:memory
-LIBS:microchip
-LIBS:microchip_dspic33dsc
-LIBS:microchip_pic10mcu
-LIBS:microchip_pic12mcu
-LIBS:microchip_pic16mcu
-LIBS:microchip_pic18mcu
-LIBS:microchip_pic24mcu
-LIBS:microchip_pic32mcu
-LIBS:microcontrollers
-LIBS:modules
-LIBS:motor_drivers
-LIBS:motorola
-LIBS:motors
-LIBS:msp430
-LIBS:nordicsemi
-LIBS:nxp
-LIBS:nxp_armmcu
-LIBS:onsemi
-LIBS:opto
-LIBS:Oscillators
-LIBS:philips
-LIBS:power
-LIBS:powerint
-LIBS:Power_Management
-LIBS:pspice
-LIBS:references
-LIBS:regul
-LIBS:relays
-LIBS:rfcom
-LIBS:RFSolutions
-LIBS:sensors
-LIBS:silabs
-LIBS:siliconi
-LIBS:stm8
-LIBS:stm32
-LIBS:supertex
-LIBS:switches
-LIBS:texas
-LIBS:transf
-LIBS:transistors
-LIBS:triac_thyristor
-LIBS:ttl_ieee
-LIBS:valves
-LIBS:video
-LIBS:wiznet
-LIBS:Worldsemi
-LIBS:Xicor
-LIBS:xilinx
-LIBS:zetex
-LIBS:Zilog
-LIBS:bd9e302efj
-LIBS:psmn1
-LIBS:tmc2130
+EESchema Schematic File Version 4
 LIBS:schematic-cache
-EELAYER 25 0
+EELAYER 26 0
 EELAYER END
 $Descr A4 11693 8268
@@
 $EndDescr
 $Comp
-L R R66
+L Device:R R66
 U 1 1 59EDEBD6
 P 3350 2350
+AR Path="/59EDEBD6" Ref="R66"  Part="1"
+AR Path="/59EDEA0E/59EDEBD6" Ref="R66"  Part="1"
 F 0 "R66" V 3430 2350 50  0000 C CNN
 F 1 "1.6K" V 3350 2350 50  0000 C CNN
@@
 $EndComp
 $Comp
-L R R69
+L Device:R R69
 U 1 1 59EDEC86
 P 3850 2350
+AR Path="/59EDEC86" Ref="R69"  Part="1"
+AR Path="/59EDEA0E/59EDEC86" Ref="R69"  Part="1"
 F 0 "R69" V 3930 2350 50  0000 C CNN
 F 1 "1.6K" V 3850 2350 50  0000 C CNN
@@
 $EndComp
 $Comp
-L C C100
+L Device:C C100
 U 1 1 59EDECB4
 P 3600 2600
+AR Path="/59EDECB4" Ref="C100"  Part="1"
+AR Path="/59EDEA0E/59EDECB4" Ref="C100"  Part="1"
 F 0 "C100" H 3625 2700 50  0000 L CNN
 F 1 "1uF" H 3625 2500 50  0000 L CNN
@@
 $EndComp
 $Comp
-L C C103
+L Device:C C103
 U 1 1 59EDECF2
 P 4100 2600
+AR Path="/59EDECF2" Ref="C103"  Part="1"
+AR Path="/59EDEA0E/59EDECF2" Ref="C103"  Part="1"
 F 0 "C103" H 4125 2700 50  0000 L CNN
 F 1 "1uF" H 4125 2500 50  0000 L CNN
@@
 $EndComp
 $Comp
-L R R72
+L Device:R R72
 U 1 1 59EDED24
 P 4350 2600
+AR Path="/59EDED24" Ref="R72"  Part="1"
+AR Path="/59EDEA0E/59EDED24" Ref="R72"  Part="1"
 F 0 "R72" V 4430 2600 50  0000 C CNN
 F 1 "10K" V 4350 2600 50  0000 C CNN
@@
 Connection ~ 4100 2350
 $Comp
-L GND #PWR147
+L power:GND #PWR0147
 U 1 1 59EDEDD1
 P 3600 2750
-F 0 "#PWR147" H 3600 2500 50  0001 C CNN
+F 0 "#PWR0147" H 3600 2500 50  0001 C CNN
 F 1 "GND" H 3600 2600 50  0000 C CNN
 F 2 "" H 3600 2750 50  0001 C CNN
@@
 $EndComp
 $Comp
-L GND #PWR150
+L power:GND #PWR0150
 U 1 1 59EDEDF4
 P 4100 2750
-F 0 "#PWR150" H 4100 2500 50  0001 C CNN
+F 0 "#PWR0150" H 4100 2500 50  0001 C CNN
 F 1 "GND" H 4100 2600 50  0000 C CNN
 F 2 "" H 4100 2750 50  0001 C CNN
@@
 $EndComp
 $Comp
-L GND #PWR153
+L power:GND #PWR0153
 U 1 1 59EDEE17
 P 4350 2750
-F 0 "#PWR153" H 4350 2500 50  0001 C CNN
+F 0 "#PWR0153" H 4350 2500 50  0001 C CNN
 F 1 "GND" H 4350 2600 50  0000 C CNN
 F 2 "" H 4350 2750 50  0001 C CNN
@@
 Connection ~ 4350 2350
 $Comp
-L R R67
+L Device:R R67
 U 1 1 59EE0353
 P 3350 3050
+AR Path="/59EE0353" Ref="R67"  Part="1"
+AR Path="/59EDEA0E/59EE0353" Ref="R67"  Part="1"
 F 0 "R67" V 3430 3050 50  0000 C CNN
 F 1 "1.6K" V 3350 3050 50  0000 C CNN
@@
 $EndComp
 $Comp
-L R R70
+L Device:R R70
 U 1 1 59EE0359
 P 3850 3050
+AR Path="/59EE0359" Ref="R70"  Part="1"
+AR Path="/59EDEA0E/59EE0359" Ref="R70"  Part="1"
 F 0 "R70" V 3930 3050 50  0000 C CNN
 F 1 "1.6K" V 3850 3050 50  0000 C CNN
@@
 $EndComp
 $Comp
-L C C101
+L Device:C C101
 U 1 1 59EE035F
 P 3600 3300
+AR Path="/59EE035F" Ref="C101"  Part="1"
+AR Path="/59EDEA0E/59EE035F" Ref="C101"  Part="1"
 F 0 "C101" H 3625 3400 50  0000 L CNN
 F 1 "1uF" H 3625 3200 50  0000 L CNN
@@
 $EndComp
 $Comp
-L C C104
+L Device:C C104
 U 1 1 59EE0365
 P 4100 3300
+AR Path="/59EE0365" Ref="C104"  Part="1"
+AR Path="/59EDEA0E/59EE0365" Ref="C104"  Part="1"
 F 0 "C104" H 4125 3400 50  0000 L CNN
 F 1 "1uF" H 4125 3200 50  0000 L CNN
@@
 $EndComp
 $Comp
-L R R73
+L Device:R R73
 U 1 1 59EE036B
 P 4350 3300
+AR Path="/59EE036B" Ref="R73"  Part="1"
+AR Path="/59EDEA0E/59EE036B" Ref="R73"  Part="1"
 F 0 "R73" V 4430 3300 50  0000 C CNN
 F 1 "10K" V 4350 3300 50  0000 C CNN
@@
 Connection ~ 4100 3050
 $Comp
-L GND #PWR148
+L power:GND #PWR0148
 U 1 1 59EE0378
 P 3600 3450
-F 0 "#PWR148" H 3600 3200 50  0001 C CNN
+F 0 "#PWR0148" H 3600 3200 50  0001 C CNN
 F 1 "GND" H 3600 3300 50  0000 C CNN
 F 2 "" H 3600 3450 50  0001 C CNN
@@
 $EndComp
 $Comp
-L GND #PWR151
+L power:GND #PWR0151
 U 1 1 59EE037E
 P 4100 3450
-F 0 "#PWR151" H 4100 3200 50  0001 C CNN
+F 0 "#PWR0151" H 4100 3200 50  0001 C CNN
 F 1 "GND" H 4100 3300 50  0000 C CNN
 F 2 "" H 4100 3450 50  0001 C CNN
@@
 $EndComp
 $Comp
-L GND #PWR154
+L power:GND #PWR0154
 U 1 1 59EE0384
 P 4350 3450
-F 0 "#PWR154" H 4350 3200 50  0001 C CNN
+F 0 "#PWR0154" H 4350 3200 50  0001 C CNN
 F 1 "GND" H 4350 3300 50  0000 C CNN
 F 2 "" H 4350 3450 50  0001 C CNN
@@
 Connection ~ 4350 3050
 $Comp
-L R R68
+L Device:R R68
 U 1 1 59EE04D7
 P 3350 3750
+AR Path="/59EE04D7" Ref="R68"  Part="1"
+AR Path="/59EDEA0E/59EE04D7" Ref="R68"  Part="1"
 F 0 "R68" V 3430 3750 50  0000 C CNN
 F 1 "1.6K" V 3350 3750 50  0000 C CNN
@@
 $EndComp
 $Comp
-L R R71
+L Device:R R71
 U 1 1 59EE04DD
 P 3850 3750
+AR Path="/59EE04DD" Ref="R71"  Part="1"
+AR Path="/59EDEA0E/59EE04DD" Ref="R71"  Part="1"
 F 0 "R71" V 3930 3750 50  0000 C CNN
 F 1 "1.6K" V 3850 3750 50  0000 C CNN
@@
 $EndComp
 $Comp
-L C C102
+L Device:C C102
 U 1 1 59EE04E3
 P 3600 4000
+AR Path="/59EE04E3" Ref="C102"  Part="1"
+AR Path="/59EDEA0E/59EE04E3" Ref="C102"  Part="1"
 F 0 "C102" H 3625 4100 50  0000 L CNN
 F 1 "1uF" H 3625 3900 50  0000 L CNN
@@
 $EndComp
 $Comp
-L C C105
+L Device:C C105
 U 1 1 59EE04E9
 P 4100 4000
+AR Path="/59EE04E9" Ref="C105"  Part="1"
+AR Path="/59EDEA0E/59EE04E9" Ref="C105"  Part="1"
 F 0 "C105" H 4125 4100 50  0000 L CNN
 F 1 "1uF" H 4125 3900 50  0000 L CNN
@@
 $EndComp
 $Comp
-L R R74
+L Device:R R74
 U 1 1 59EE04EF
 P 4350 4000
+AR Path="/59EE04EF" Ref="R74"  Part="1"
+AR Path="/59EDEA0E/59EE04EF" Ref="R74"  Part="1"
 F 0 "R74" V 4430 4000 50  0000 C CNN
 F 1 "10K" V 4350 4000 50  0000 C CNN
@@
 Connection ~ 4100 3750
 $Comp
-L GND #PWR149
+L power:GND #PWR0149
 U 1 1 59EE04FC
 P 3600 4150
-F 0 "#PWR149" H 3600 3900 50  0001 C CNN
+F 0 "#PWR0149" H 3600 3900 50  0001 C CNN
 F 1 "GND" H 3600 4000 50  0000 C CNN
 F 2 "" H 3600 4150 50  0001 C CNN
@@
 $EndComp
 $Comp
-L GND #PWR152
+L power:GND #PWR0152
 U 1 1 59EE0502
 P 4100 4150
-F 0 "#PWR152" H 4100 3900 50  0001 C CNN
+F 0 "#PWR0152" H 4100 3900 50  0001 C CNN
 F 1 "GND" H 4100 4000 50  0000 C CNN
 F 2 "" H 4100 4150 50  0001 C CNN
@@
 $EndComp
 $Comp
-L GND #PWR155
+L power:GND #PWR0155
 U 1 1 59EE0508
 P 4350 4150
-F 0 "#PWR155" H 4350 3900 50  0001 C CNN
+F 0 "#PWR0155" H 4350 3900 50  0001 C CNN
 F 1 "GND" H 4350 4000 50  0000 C CNN
 F 2 "" H 4350 4150 50  0001 C CNN

Commit message: Revert "Updated to kicad 5.0.0"
This reverts commit 6c14fa6c8e6361c9b9ee4065803a5a63755fc6a7.
Parts:
- C100, C101, C102, C103, C104, C105: symbol Device:C -> C
- R66, R67, R68, R69, R70, R71, R72, R73, R74: symbol Device:R -> R
Changed lines of the file:
@@
-EESchema Schematic File Version 4
+EESchema Schematic File Version 2
+LIBS:74xgxx
+LIBS:74xx
+LIBS:ac-dc
+LIBS:actel
+LIBS:adc-dac
+LIBS:allegro
+LIBS:Altera
+LIBS:analog_devices
+LIBS:analog_switches
+LIBS:atmel
+LIBS:audio
+LIBS:battery_management
+LIBS:bbd
+LIBS:bosch
+LIBS:brooktre
+LIBS:cmos4000
+LIBS:cmos_ieee
+LIBS:conn
+LIBS:contrib
+LIBS:cypress
+LIBS:dc-dc
+LIBS:device
+LIBS:digital-audio
+LIBS:diode
+LIBS:display
+LIBS:dsp
+LIBS:elec-unifil
+LIBS:ESD_Protection
+LIBS:ftdi
+LIBS:gennum
+LIBS:graphic_symbols
+LIBS:hc11
+LIBS:infineon
+LIBS:intel
+LIBS:interface
+LIBS:intersil
+LIBS:ir
+LIBS:Lattice
+LIBS:leds
+LIBS:LEM
+LIBS:linear
+LIBS:logic_programmable
+LIBS:maxim
+LIBS:mechanical
+LIBS:memory
+LIBS:microchip
+LIBS:microchip_dspic33dsc
+LIBS:microchip_pic10mcu
+LIBS:microchip_pic12mcu
+LIBS:microchip_pic16mcu
+LIBS:microchip_pic18mcu
+LIBS:microchip_pic24mcu
+LIBS:microchip_pic32mcu
+LIBS:microcontrollers
+LIBS:modules
+LIBS:motor_drivers
+LIBS:motorola
+LIBS:motors
+LIBS:msp430
+LIBS:nordicsemi
+LIBS:nxp
+LIBS:nxp_armmcu
+LIBS:onsemi
+LIBS:opto
+LIBS:Oscillators
+LIBS:philips
+LIBS:power
+LIBS:powerint
+LIBS:Power_Management
+LIBS:pspice
+LIBS:references
+LIBS:regul
+LIBS:relays
+LIBS:rfcom
+LIBS:RFSolutions
+LIBS:sensors
+LIBS:silabs
+LIBS:siliconi
+LIBS:stm8
+LIBS:stm32
+LIBS:supertex
+LIBS:switches
+LIBS:texas
+LIBS:transf
+LIBS:transistors
+LIBS:triac_thyristor
+LIBS:ttl_ieee
+LIBS:valves
+LIBS:video
+LIBS:wiznet
+LIBS:Worldsemi
+LIBS:Xicor
+LIBS:xilinx
+LIBS:zetex
+LIBS:Zilog
+LIBS:bd9e302efj
+LIBS:psmn1
+LIBS:tmc2130
 LIBS:schematic-cache
-EELAYER 26 0
+EELAYER 25 0
 EELAYER END
 $Descr A4 11693 8268
@@
 $EndDescr
 $Comp
-L Device:R R66
+L R R66
 U 1 1 59EDEBD6
 P 3350 2350
-AR Path="/59EDEBD6" Ref="R66"  Part="1"
-AR Path="/59EDEA0E/59EDEBD6" Ref="R66"  Part="1"
 F 0 "R66" V 3430 2350 50  0000 C CNN
 F 1 "1.6K" V 3350 2350 50  0000 C CNN
@@
 $EndComp
 $Comp
-L Device:R R69
+L R R69
 U 1 1 59EDEC86
 P 3850 2350
-AR Path="/59EDEC86" Ref="R69"  Part="1"
-AR Path="/59EDEA0E/59EDEC86" Ref="R69"  Part="1"
 F 0 "R69" V 3930 2350 50  0000 C CNN
 F 1 "1.6K" V 3850 2350 50  0000 C CNN
@@
 $EndComp
 $Comp
-L Device:C C100
+L C C100
 U 1 1 59EDECB4
 P 3600 2600
-AR Path="/59EDECB4" Ref="C100"  Part="1"
-AR Path="/59EDEA0E/59EDECB4" Ref="C100"  Part="1"
 F 0 "C100" H 3625 2700 50  0000 L CNN
 F 1 "1uF" H 3625 2500 50  0000 L CNN
@@
 $EndComp
 $Comp
-L Device:C C103
+L C C103
 U 1 1 59EDECF2
 P 4100 2600
-AR Path="/59EDECF2" Ref="C103"  Part="1"
-AR Path="/59EDEA0E/59EDECF2" Ref="C103"  Part="1"
 F 0 "C103" H 4125 2700 50  0000 L CNN
 F 1 "1uF" H 4125 2500 50  0000 L CNN
@@
 $EndComp
 $Comp
-L Device:R R72
+L R R72
 U 1 1 59EDED24
 P 4350 2600
-AR Path="/59EDED24" Ref="R72"  Part="1"
-AR Path="/59EDEA0E/59EDED24" Ref="R72"  Part="1"
 F 0 "R72" V 4430 2600 50  0000 C CNN
 F 1 "10K" V 4350 2600 50  0000 C CNN
@@
 Connection ~ 4100 2350
 $Comp
-L power:GND #PWR0147
+L GND #PWR147
 U 1 1 59EDEDD1
 P 3600 2750
-F 0 "#PWR0147" H 3600 2500 50  0001 C CNN
+F 0 "#PWR147" H 3600 2500 50  0001 C CNN
 F 1 "GND" H 3600 2600 50  0000 C CNN
 F 2 "" H 3600 2750 50  0001 C CNN
@@
 $EndComp
 $Comp
-L power:GND #PWR0150
+L GND #PWR150
 U 1 1 59EDEDF4
 P 4100 2750
-F 0 "#PWR0150" H 4100 2500 50  0001 C CNN
+F 0 "#PWR150" H 4100 2500 50  0001 C CNN
 F 1 "GND" H 4100 2600 50  0000 C CNN
 F 2 "" H 4100 2750 50  0001 C CNN
@@
 $EndComp
 $Comp
-L power:GND #PWR0153
+L GND #PWR153
 U 1 1 59EDEE17
 P 4350 2750
-F 0 "#PWR0153" H 4350 2500 50  0001 C CNN
+F 0 "#PWR153" H 4350 2500 50  0001 C CNN
 F 1 "GND" H 4350 2600 50  0000 C CNN
 F 2 "" H 4350 2750 50  0001 C CNN
@@
 Connection ~ 4350 2350
 $Comp
-L Device:R R67
+L R R67
 U 1 1 59EE0353
 P 3350 3050
-AR Path="/59EE0353" Ref="R67"  Part="1"
-AR Path="/59EDEA0E/59EE0353" Ref="R67"  Part="1"
 F 0 "R67" V 3430 3050 50  0000 C CNN
 F 1 "1.6K" V 3350 3050 50  0000 C CNN
@@
 $EndComp
 $Comp
-L Device:R R70
+L R R70
 U 1 1 59EE0359
 P 3850 3050
-AR Path="/59EE0359" Ref="R70"  Part="1"
-AR Path="/59EDEA0E/59EE0359" Ref="R70"  Part="1"
 F 0 "R70" V 3930 3050 50  0000 C CNN
 F 1 "1.6K" V 3850 3050 50  0000 C CNN
@@
 $EndComp
 $Comp
-L Device:C C101
+L C C101
 U 1 1 59EE035F
 P 3600 3300
-AR Path="/59EE035F" Ref="C101"  Part="1"
-AR Path="/59EDEA0E/59EE035F" Ref="C101"  Part="1"
 F 0 "C101" H 3625 3400 50  0000 L CNN
 F 1 "1uF" H 3625 3200 50  0000 L CNN
@@
 $EndComp
 $Comp
-L Device:C C104
+L C C104
 U 1 1 59EE0365
 P 4100 3300
-AR Path="/59EE0365" Ref="C104"  Part="1"
-AR Path="/59EDEA0E/59EE0365" Ref="C104"  Part="1"
 F 0 "C104" H 4125 3400 50  0000 L CNN
 F 1 "1uF" H 4125 3200 50  0000 L CNN
@@
 $EndComp
 $Comp
-L Device:R R73
+L R R73
 U 1 1 59EE036B
 P 4350 3300
-AR Path="/59EE036B" Ref="R73"  Part="1"
-AR Path="/59EDEA0E/59EE036B" Ref="R73"  Part="1"
 F 0 "R73" V 4430 3300 50  0000 C CNN
 F 1 "10K" V 4350 3300 50  0000 C CNN
@@
 Connection ~ 4100 3050
 $Comp
-L power:GND #PWR0148
+L GND #PWR148
 U 1 1 59EE0378
 P 3600 3450
-F 0 "#PWR0148" H 3600 3200 50  0001 C CNN
+F 0 "#PWR148" H 3600 3200 50  0001 C CNN
 F 1 "GND" H 3600 3300 50  0000 C CNN
 F 2 "" H 3600 3450 50  0001 C CNN
@@
 $EndComp
 $Comp
-L power:GND #PWR0151
+L GND #PWR151
 U 1 1 59EE037E
 P 4100 3450
-F 0 "#PWR0151" H 4100 3200 50  0001 C CNN
+F 0 "#PWR151" H 4100 3200 50  0001 C CNN
 F 1 "GND" H 4100 3300 50  0000 C CNN
 F 2 "" H 4100 3450 50  0001 C CNN
@@
 $EndComp
 $Comp
-L power:GND #PWR0154
+L GND #PWR154
 U 1 1 59EE0384
 P 4350 3450
-F 0 "#PWR0154" H 4350 3200 50  0001 C CNN
+F 0 "#PWR154" H 4350 3200 50  0001 C CNN
 F 1 "GND" H 4350 3300 50  0000 C CNN
 F 2 "" H 4350 3450 50  0001 C CNN
@@
 Connection ~ 4350 3050
 $Comp
-L Device:R R68
+L R R68
 U 1 1 59EE04D7
 P 3350 3750
-AR Path="/59EE04D7" Ref="R68"  Part="1"
-AR Path="/59EDEA0E/59EE04D7" Ref="R68"  Part="1"
 F 0 "R68" V 3430 3750 50  0000 C CNN
 F 1 "1.6K" V 3350 3750 50  0000 C CNN
@@
 $EndComp
 $Comp
-L Device:R R71
+L R R71
 U 1 1 59EE04DD
 P 3850 3750
-AR Path="/59EE04DD" Ref="R71"  Part="1"
-AR Path="/59EDEA0E/59EE04DD" Ref="R71"  Part="1"
 F 0 "R71" V 3930 3750 50  0000 C CNN
 F 1 "1.6K" V 3850 3750 50  0000 C CNN
@@
 $EndComp
 $Comp
-L Device:C C102
+L C C102
 U 1 1 59EE04E3
 P 3600 4000
-AR Path="/59EE04E3" Ref="C102"  Part="1"
-AR Path="/59EDEA0E/59EE04E3" Ref="C102"  Part="1"
 F 0 "C102" H 3625 4100 50  0000 L CNN
 F 1 "1uF" H 3625 3900 50  0000 L CNN
@@
 $EndComp
 $Comp
-L Device:C C105
+L C C105
 U 1 1 59EE04E9
 P 4100 4000
-AR Path="/59EE04E9" Ref="C105"  Part="1"
-AR Path="/59EDEA0E/59EE04E9" Ref="C105"  Part="1"
 F 0 "C105" H 4125 4100 50  0000 L CNN
 F 1 "1uF" H 4125 3900 50  0000 L CNN
@@
 $EndComp
 $Comp
-L Device:R R74
+L R R74
 U 1 1 59EE04EF
 P 4350 4000
-AR Path="/59EE04EF" Ref="R74"  Part="1"
-AR Path="/59EDEA0E/59EE04EF" Ref="R74"  Part="1"
 F 0 "R74" V 4430 4000 50  0000 C CNN
 F 1 "10K" V 4350 4000 50  0000 C CNN
@@
 Connection ~ 4100 3750
 $Comp
-L power:GND #PWR0149
+L GND #PWR149
 U 1 1 59EE04FC
 P 3600 4150
-F 0 "#PWR0149" H 3600 3900 50  0001 C CNN
+F 0 "#PWR149" H 3600 3900 50  0001 C CNN
 F 1 "GND" H 3600 4000 50  0000 C CNN
 F 2 "" H 3600 4150 50  0001 C CNN
@@
 $EndComp
 $Comp
-L power:GND #PWR0152
+L GND #PWR152
 U 1 1 59EE0502
 P 4100 4150
-F 0 "#PWR0152" H 4100 3900 50  0001 C CNN
+F 0 "#PWR152" H 4100 3900 50  0001 C CNN
 F 1 "GND" H 4100 4000 50  0000 C CNN
 F 2 "" H 4100 4150 50  0001 C CNN
@@
 $EndComp
 $Comp
-L power:GND #PWR0155
+L GND #PWR155
 U 1 1 59EE0508
 P 4350 4150
-F 0 "#PWR0155" H 4350 3900 50  0001 C CNN
+F 0 "#PWR155" H 4350 3900 50  0001 C CNN
 F 1 "GND" H 4350 4000 50  0000 C CNN
 F 2 "" H 4350 4150 50  0001 C CNN
